File: Hardware/Chancey-board_modular-AA/Chancey-board_modular-AA.kicad_pcb (KiCad board)
At the start: 2 copper layers, 373.9 x 123.8 mm, 194 parts, among them J1 QWIIC, U1 Hall_Sensor, U10 Hall_Sensor, U11 Hall_Sensor, U12 Hall_Sensor, U13 Hall_Sensor, U14 Hall_Sensor, U15 Hall_Sensor, U16 Hall_Sensor, U17 Hall_Sensor, U18 Hall_Sensor, U19 Hall_Sensor, U20 Hall_Sensor, U21 Hall_Sensor, U22 Hall_Sensor, U23 Hall_Sensor, U24 Hall_Sensor, U25 Hall_Sensor, U26 Hall_Sensor, U27 Hall_Sensor, U28 Hall_Sensor, U29 Hall_Sensor, U30 Hall_Sensor, U31 Hall_Sensor, U32 Hall_Sensor, U33 Hall_Sensor, U34 Hall_Sensor, U35 Hall_Sensor, U36 Hall_Sensor, U37 Hall_Sensor, U38 Hall_Sensor, U39 Hall_Sensor, U40 Hall_Sensor, U41 Hall_Sensor, U42 Hall_Sensor, U43 Hall_Sensor, U44 Hall_Sensor, U45 Hall_Sensor, U46 Hall_Sensor, U47 Hall_Sensor, U48 Hall_Sensor, U49 Hall_Sensor, U50 Hall_Sensor, U51 Hall_Sensor, U52 Hall_Sensor, U53 Hall_Sensor, U54 Hall_Sensor, U55 Hall_Sensor, U56 Hall_Sensor, U57 Hall_Sensor, U58 Hall_Sensor, U59 Hall_Sensor, U6 BlackPill_STLINK, U60 Hall_Sensor, U61 Hall_Sensor, U62 Hall_Sensor, U63 Hall_Sensor, U64 Hall_Sensor, U65 Hall_Sensor, U66 Hall_Sensor, U67 Hall_Sensor, U68 Hall_Sensor, U69 Hall_Sensor, U7 Hall_Sensor, U70 Hall_Sensor, U71 Hall_Sensor, U72 Hall_Sensor, U73 Hall_Sensor, U74 Hall_Sensor, U75 Hall_Sensor, U76 Hall_Sensor, U8 Hall_Sensor, U9 Hall_Sensor

Commit message: Changed many global labels to hierarchical and local labels.
Parts:
- added AM5:1: F1, Chancey_modular:VoidSwitch_1u_SMD, F.Cu at (238.1, 199.9)
- added AM5:10: F10, Chancey_modular:VoidSwitch_1u_SMD, F.Cu at (418.7, 198.1)
- added AM5:11: F11, Chancey_modular:VoidSwitch_1u_SMD, F.Cu at (438.9, 198.1)
- added AM5:12: F12, Chancey_modular:VoidSwitch_1u_SMD, F.Cu at (459.1, 198.1)
- added AM5:13: END, Chancey_modular:VoidSwitch_1u_SMD, F.Cu at (652.1, 198.8)
- added AM5:14: Insert, Chancey_modular:VoidSwitch_1u_SMD, F.Cu at (652.1, 219.0)
- added AM5:15: Home, Chancey_modular:VoidSwitch_1u_SMD, F.Cu at (652.1, 239.2)
- added AM5:2: F2, Chancey_modular:VoidSwitch_1u_SMD, F.Cu at (258.3, 199.9)
- added AM5:3: F3, Chancey_modular:VoidSwitch_1u_SMD, F.Cu at (278.5, 199.9)
- added AM5:4: F4, Chancey_modular:VoidSwitch_1u_SMD, F.Cu at (298.7, 199.9)
- added AM5:5: F5, Chancey_modular:VoidSwitch_1u_SMD, F.Cu at (318.9, 199.9)
- added AM5:6: F6, Chancey_modular:VoidSwitch_1u_SMD, F.Cu at (339.1, 199.9)
- added AM5:7: F7, Chancey_modular:VoidSwitch_1u_SMD, F.Cu at (358.1, 198.1)
- added AM5:8: F8, Chancey_modular:VoidSwitch_1u_SMD, F.Cu at (378.3, 198.1)
- added AM5:9: F9, Chancey_modular:VoidSwitch_1u_SMD, F.Cu at (398.5, 198.1)
- added AM6: CD74HC4067SM, Package_SO:SSOP-24_5.3x8.2mm_P0.65mm, F.Cu at (620.8, 250.4)
- added AM6:0: Pg.Up, Chancey_modular:VoidSwitch_1u_SMD, F.Cu at (652.1, 259.4)
- added AM6:1: DELETE, Chancey_modular:VoidSwitch_1u_SMD, F.Cu at (652.1, 279.6)
- added AM6:2: Pg.Dn, Chancey_modular:VoidSwitch_1u_SMD, F.Cu at (652.1, 299.8)
- added AM6:3: Prt.Scrn, Chancey_modular:VoidSwitch_1u_SMD, F.Cu at (672.3, 198.8)
- added AM6:4: Scrol.lk, Chancey_modular:VoidSwitch_1u_SMD, F.Cu at (672.3, 219.0)
- added AM6:5: Pause, Chancey_modular:VoidSwitch_1u_SMD, F.Cu at (672.3, 239.2)
- added AM7: CD74HC4067SM, Package_SO:SSOP-24_5.3x8.2mm_P0.65mm, F.Cu at (676.8, 250.4)
- added R8: 2k2, Resistor_SMD:R_0402_1005Metric, F.Cu at (226.5, 241.6)
- added R9: 2k2, Resistor_SMD:R_0402_1005Metric, F.Cu at (226.5, 243.6)
- added U0: Hall_Sensor, Package_TO_SOT_SMD:SOT-23, F.Cu at (429.9, 202.6)
- added U2: Hall_Sensor, Package_TO_SOT_SMD:SOT-23, F.Cu at (559.8, 218.6)
- added U3: Hall_Sensor, Package_TO_SOT_SMD:SOT-23, F.Cu at (562.9, 221.8)
- added U4: Hall_Sensor, Package_TO_SOT_SMD:SOT-23, F.Cu at (566.1, 224.9)
- added U5: Hall_Sensor, Package_TO_SOT_SMD:SOT-23, F.Cu at (569.2, 228.0)
- added UTab1: Hall_Sensor, Package_TO_SOT_SMD:SOT-23, F.Cu at (572.4, 231.2)
- added U_BP1: BlackPill_STLINK, Chancey_modular:BlackPill_STLINK, F.Cu at (357.2, 197.4)
- added U_BS1: Hall_Sensor, Package_TO_SOT_SMD:SOT-23, F.Cu at (560.1, 212.0)
- added U_BS34: Hall_Sensor, Package_TO_SOT_SMD:SOT-23, F.Cu at (563.2, 215.1)
- added U_DE1: Hall_Sensor, Package_TO_SOT_SMD:SOT-23, F.Cu at (605.2, 276.5)
- added U_Di1: Hall_Sensor, Package_TO_SOT_SMD:SOT-23, F.Cu at (608.3, 279.7)
- added U_E24: Hall_Sensor, Package_TO_SOT_SMD:SOT-23, F.Cu at (569.5, 221.4)
- added U_E7: Hall_Sensor, Package_TO_SOT_SMD:SOT-23, F.Cu at (566.4, 218.3)
- added U_EN1: Hall_Sensor, Package_TO_SOT_SMD:SOT-23, F.Cu at (611.5, 282.8)
- added U_I29: Hall_Sensor, Package_TO_SOT_SMD:SOT-23, F.Cu at (572.7, 224.6)
- added U_In1: Hall_Sensor, Package_TO_SOT_SMD:SOT-23, F.Cu at (614.6, 286.0)
- added U_LB32: Hall_Sensor, Package_TO_SOT_SMD:SOT-23, F.Cu at (575.8, 227.7)
- added U_LM1: Hall_Sensor, Package_TO_SOT_SMD:SOT-23, F.Cu at (563.5, 208.5)
- added U_LP1: Hall_Sensor, Package_TO_SOT_SMD:SOT-23, F.Cu at (566.7, 211.7)
- added U_ND1: Hall_Sensor, Package_TO_SOT_SMD:SOT-23, F.Cu at (617.8, 289.1)
- added U_NL1: Hall_Sensor, Package_TO_SOT_SMD:SOT-23, F.Cu at (608.6, 273.1)
- added U_NP0: Hall_Sensor, Package_TO_SOT_SMD:SOT-23, F.Cu at (611.8, 276.2)
- added U_NP1: Hall_Sensor, Package_TO_SOT_SMD:SOT-23, F.Cu at (614.9, 279.4)
- added U_NP10: Hall_Sensor, Package_TO_SOT_SMD:SOT-23, F.Cu at (618.7, 269.3)
- added U_NP2: Hall_Sensor, Package_TO_SOT_SMD:SOT-23, F.Cu at (618.1, 282.5)
- added U_NP3: Hall_Sensor, Package_TO_SOT_SMD:SOT-23, F.Cu at (621.2, 285.7)
- added U_NP4: Hall_Sensor, Package_TO_SOT_SMD:SOT-23, F.Cu at (612.1, 269.6)
- added U_NP5: Hall_Sensor, Package_TO_SOT_SMD:SOT-23, F.Cu at (615.3, 272.8)
- added U_NP6: Hall_Sensor, Package_TO_SOT_SMD:SOT-23, F.Cu at (618.4, 275.9)
- added U_NP7: Hall_Sensor, Package_TO_SOT_SMD:SOT-23, F.Cu at (621.5, 279.0)
- added U_NP8: Hall_Sensor, Package_TO_SOT_SMD:SOT-23, F.Cu at (624.7, 282.2)
- added U_NP9: Hall_Sensor, Package_TO_SOT_SMD:SOT-23, F.Cu at (615.6, 266.1)
- added U_NpT1: Hall_Sensor, Package_TO_SOT_SMD:SOT-23, F.Cu at (621.9, 272.4)
- added U_O30: Hall_Sensor, Package_TO_SOT_SMD:SOT-23, F.Cu at (569.8, 214.8)
- added U_P1: Hall_Sensor, Package_TO_SOT_SMD:SOT-23, F.Cu at (625.0, 275.6)
- added U_P31: Hall_Sensor, Package_TO_SOT_SMD:SOT-23, F.Cu at (573.0, 218.0)
- added U_PD1: Hall_Sensor, Package_TO_SOT_SMD:SOT-23, F.Cu at (628.2, 278.7)
- added U_PS1: Hall_Sensor, Package_TO_SOT_SMD:SOT-23, F.Cu at (619.0, 262.7)
- added U_PU1: Hall_Sensor, Package_TO_SOT_SMD:SOT-23, F.Cu at (622.2, 265.8)
- added U_Q22: Hall_Sensor, Package_TO_SOT_SMD:SOT-23, F.Cu at (576.1, 221.1)
- added U_R25: Hall_Sensor, Package_TO_SOT_SMD:SOT-23, F.Cu at (579.3, 224.3)
- added U_RB33: Hall_Sensor, Package_TO_SOT_SMD:SOT-23, F.Cu at (567.0, 205.1)
- added U_RM1: Hall_Sensor, Package_TO_SOT_SMD:SOT-23, F.Cu at (625.3, 269.0)
- added U_RP1: Hall_Sensor, Package_TO_SOT_SMD:SOT-23, F.Cu at (628.5, 272.1)
- added U_SL1: Hall_Sensor, Package_TO_SOT_SMD:SOT-23, F.Cu at (631.6, 275.3)
- added U_T26: Hall_Sensor, Package_TO_SOT_SMD:SOT-23, F.Cu at (570.1, 208.2)
- added U_U28: Hall_Sensor, Package_TO_SOT_SMD:SOT-23, F.Cu at (573.3, 211.4)
- added U_W23: Hall_Sensor, Package_TO_SOT_SMD:SOT-23, F.Cu at (576.4, 214.5)
- added U_Y27: Hall_Sensor, Package_TO_SOT_SMD:SOT-23, F.Cu at (579.6, 217.7)
- added U_~1: Hall_Sensor, Package_TO_SOT_SMD:SOT-23, F.Cu at (549.5, 287.2)
- AM0:0, AM0:1, AM0:15, AM3:3: footprint void_switch:VoidSwitch_1.25u_SMD -> Chancey_modular:VoidSwitch_1u_SMD
- AM0:10, AM0:11, AM0:12, AM0:13, AM0:14, AM0:2, AM0:3, AM0:4, AM0:5, AM0:6, AM0:7, AM0:8, AM0:9, AM1:0, AM1:1, AM1:10, AM1:11, AM1:12, AM1:13, AM1:14, AM1:15, AM1:3, AM1:4, AM1:5, AM1:6, AM1:7, AM1:8, AM1:9, AM2:10, AM2:11, AM2:12, AM2:13, AM2:2, AM2:3, AM2:4, AM2:5, AM2:6, AM2:7, AM2:8, AM2:9, AM3:10, AM3:11, AM3:13, AM3:14, AM3:2, AM3:4, AM3:5, AM3:6, AM3:7, AM3:8, AM3:9, AM4:0, AM4:1, AM4:12, AM4:13, AM4:14, AM4:15, AM4:3, AM4:4, AM4:5, AM4:7: footprint void_switch:VoidSwitch_1u_SMD -> Chancey_modular:VoidSwitch_1u_SMD
- AM1:2: value Fun -> Func1; footprint void_switch:VoidSwitch_1.25u_SMD -> Chancey_modular:VoidSwitch_1u_SMD
- AM2:14: value More Fun -> Func2; footprint void_switch:VoidSwitch_1.25u_SMD -> Chancey_modular:VoidSwitch_1u_SMD
- AM3:1: value Slash -> Quest; footprint void_switch:VoidSwitch_1u_SMD -> Chancey_modular:VoidSwitch_1u_SMD
- AM3:12: value Quot -> Fslash; footprint void_switch:VoidSwitch_1u_SMD -> Chancey_modular:VoidSwitch_1u_SMD
- AM4:6: value BS -> Bspace; footprint void_switch:VoidSwitch_1u_SMD -> Chancey_modular:VoidSwitch_1u_SMD
- U6: value BlackPill_STLINK -> Hall_Sensor; footprint blackpill:BlackPill_STLINK -> Package_TO_SOT_SMD:SOT-23
- moved U_F1 325.5 mm to (229.3, 204.1), turned to 45 degrees
- moved U_F2 320.6 mm to (235.2, 203.7), turned to 45 degrees
- moved U_F3 315.5 mm to (241.5, 203.2), turned to 45 degrees
- moved U_F4 311.0 mm to (246.9, 203.1), turned to 45 degrees
- moved U_F5 305.8 mm to (252.9, 202.8), turned to 45 degrees
- moved U_F6 300.6 mm to (259.0, 202.5), turned to 45 degrees
- moved U_F7 295.9 mm to (264.7, 202.2), turned to 45 degrees
- moved U_F8 291.7 mm to (270.1, 201.9), turned to 45 degrees
- moved U_F9 287.5 mm to (275.5, 201.6), turned to 45 degrees
- moved U_F10 282.4 mm to (281.0, 201.2), turned to 45 degrees
- moved U_F11 277.9 mm to (286.5, 200.8), turned to 45 degrees
- moved U_F12 273.4 mm to (292.0, 200.5), turned to 45 degrees
- moved H4 92.0 mm to (684.9, 190.5)
- moved H8 92.0 mm to (684.9, 304.8)
- moved U1 34.6 mm to (557.6, 282.9), turned to 45 degrees
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Connections:
- net AM0:0 renamed /AM0:0
- net AM0:1 renamed /AM0:1
- net AM0:11 renamed /AM0:11
- net AM0:12 renamed /AM0:12
- net AM0:13 renamed /AM0:13
- net AM0:14 renamed /AM0:14
- net AM0:15 renamed /AM0:15
- net AM0:2 renamed /AM0:2
- net AM0:3 renamed /AM0:3
- net AM0:4 renamed /AM0:4
- net AM0:6 renamed /AM0:6
- net AM0:8 renamed /AM0:8
- net AM0:9 renamed /AM0:9
- net AM1:0 renamed /AM1:0
- net AM1:1 renamed /AM1:1
- net AM1:10 renamed /AM1:10
- net AM1:11 renamed /AM1:11
- net AM1:12 renamed /AM1:12
- net AM1:13 renamed /AM1:13
- net AM1:14 renamed /AM1:14
- net AM1:15 renamed /AM1:15
- net AM1:2 renamed /AM1:2
- net AM1:3 renamed /AM1:3
- net AM1:4 renamed /AM1:4
- net AM1:5 renamed /AM1:5
- net AM1:6 renamed /AM1:6
- net AM1:7 renamed /AM1:7
- net AM1:8 renamed /AM1:8
- net AM2:1 renamed /AM2:1
- net AM2:11 renamed /AM2:11
- net AM2:12 renamed /AM2:12
- net AM2:13 renamed /AM2:13
- net AM2:14 renamed /AM2:14
- net AM2:15 renamed /AM2:15
- net AM2:2 renamed /AM2:2
- net AM2:3 renamed /AM2:3
- net AM2:4 renamed /AM2:4
- net AM2:5 renamed /AM2:5
- net AM2:6 renamed /AM2:6
- net AM2:9 renamed /AM2:9
- net AM3:0 renamed /AM3:0
- net AM3:1 renamed /AM3:1
- net AM3:10 renamed /AM3:10
- net AM3:11 renamed /AM3:11
- net AM3:12 renamed /AM3:12
- net AM3:13 renamed /AM3:13
- net AM3:14 renamed /AM3:14
- net AM3:15 renamed /AM3:15
- net AM3:2 renamed /AM3:2
- net AM3:3 renamed /AM3:3
- net AM3:4 renamed /AM3:4
- net AM3:5 renamed /AM3:5
- net AM3:6 renamed /AM3:6
- net AM3:7 renamed /AM3:7
- net AM3:8 renamed /AM3:8
- net AM3:9 renamed /AM3:9
- net AM4:0 renamed /AM4:0
- net AM4:1 renamed /AM4:1
- net AM4:10 renamed /AM4:10
- net AM4:11 renamed /AM4:11
- net AM4:12 renamed /AM4:12
- net AM4:13 renamed /AM4:13
- net AM4:14 renamed /AM4:14
- net AM4:15 renamed /AM4:15
- net AM4:2 renamed /AM4:2
- net AM4:3 renamed /AM4:3
- net AM4:4 renamed /AM4:4
- net AM4:5 renamed /AM4:5
- net AM4:6 renamed /AM4:6
- net AM4:7 renamed /AM4:7
- net AM4:8 renamed /AM4:8
- net AM4:9 renamed /AM4:9
- net AM5:0 renamed /AM5:0
- net AM5:1 renamed /AM5:1
- net AM5:10 renamed /AM5:10
- net AM5:11 renamed /AM5:11
- net AM5:12 renamed /AM5:12
- net AM5:2 renamed /AM5:2
- net AM5:3 renamed /AM5:3
- net AM5:4 renamed /AM5:4
- net AM5:5 renamed /AM5:5
- net AM5:6 renamed /AM5:6
- net AM5:7 renamed /AM5:7
- net AM5:8 renamed /AM5:8
- net AM5:9 renamed /AM5:9
- AM0 pad 1: AM0 -> /AM0
- AM0 pad 10: SELECT0 -> /SELECT0
- AM0 pad 11: SELECT1 -> /SELECT1
- AM0 pad 13: SELECT3 -> /SELECT3
- AM0 pad 14: SELECT2 -> /SELECT2
- AM0 pad 2: AM0:7 -> /AM0:7
- AM0 pad 21: AM0:10 -> /AM0:10
- AM0 pad 4: AM0:5 -> /AM0:5
- AM1 pad 1: AM1 -> /AM1
- AM1 pad 10: SELECT0 -> /SELECT0
- AM1 pad 11: SELECT1 -> /SELECT1
- AM1 pad 13: SELECT3 -> /SELECT3
- AM1 pad 14: SELECT2 -> /SELECT2
- AM1 pad 22: AM1:9 -> /AM1:9
- AM2 pad 1: AM2 -> /AM2
- AM2 pad 10: SELECT0 -> /SELECT0
- AM2 pad 11: SELECT1 -> /SELECT1
- AM2 pad 13: SELECT3 -> /SELECT3
- AM2 pad 14: SELECT2 -> /SELECT2
- AM2 pad 2: AM2:7 -> /AM2:7
- AM2 pad 21: AM2:10 -> /AM2:10
- AM2 pad 23: AM2:8 -> /AM2:8
- AM2 pad 9: AM2:0 -> /AM2:0
- AM3 pad 1: AM3 -> /AM3
- AM3 pad 10: SELECT0 -> /SELECT0
- AM3 pad 11: SELECT1 -> /SELECT1
- AM3 pad 13: SELECT3 -> /SELECT3
- AM3 pad 14: SELECT2 -> /SELECT2
- AM4 pad 1: AM4 -> /AM4
- AM4 pad 10: SELECT0 -> /SELECT0
- AM4 pad 11: SELECT1 -> /SELECT1
- AM4 pad 13: SELECT3 -> /SELECT3
- AM4 pad 14: SELECT2 -> /SELECT2
- AM5 pad 1: AM5 -> /AM5
- AM5 pad 10: SELECT0 -> /SELECT0
- AM5 pad 11: SELECT1 -> /SELECT1
- AM5 pad 13: SELECT3 -> /SELECT3
- AM5 pad 14: SELECT2 -> /SELECT2
- AM5 pad 16: AM5:15 -> /AM5:15
- AM5 pad 17: AM5:14 -> /AM5:14
- AM5 pad 18: AM5:13 -> /AM5:13
- U1 pad 2: AM2:0 -> /AM0:7
- U13 pad 2: AM1:9 -> /AM1:9
- U14 pad 2: AM2:7 -> /AM2:7
- U15 pad 2: AM2:8 -> /AM2:8
- U16 pad 2: AM2:10 -> /AM2:10
- U6 pad 1: SELECT2 -> +3.3V
- U6 pad 2: PB13_SCK2 -> /AM1:9
- U6 pad 3: PB14_MISO2 -> GND
- U7 pad 2: AM0:5 -> /AM2:7
- U8 pad 2: AM0:7 -> /AM2:8
- U9 pad 2: AM0:10 -> /AM2:10
- U_H1 pad 2: AM5:14 -> /AM5:15
Routing:
- net SELECT2: track 310.4 -> 0.00 mm, vias 7 -> 0
- net /SELECT2: track 0.00 -> 310.4 mm, vias 0 -> 7
- net SELECT1: track 309.5 -> 0.00 mm, vias 6 -> 0
- net /SELECT1: track 0.00 -> 309.5 mm, vias 0 -> 6
- net SELECT3: track 307.8 -> 0.00 mm, vias 7 -> 0
- net /SELECT3: track 0.00 -> 307.8 mm, vias 0 -> 7
- net SELECT0: track 292.7 -> 0.00 mm, vias 6 -> 0
- net /SELECT0: track 0.00 -> 292.7 mm, vias 0 -> 6
- net AM4: track 166.3 -> 0.00 mm
- net /AM4: track 0.00 -> 166.3 mm
- net AM3: track 121.1 -> 0.00 mm
- net /AM3: track 0.00 -> 121.1 mm
- net AM0: track 107.3 -> 0.00 mm
- net /AM0: track 0.00 -> 107.3 mm
- net AM2: track 65.7 -> 0.00 mm
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Other:
- board size 373.9 x 123.8 mm -> 465.9 x 123.8 mm
